Commit message: feat: rail calibration with limit switches, 71.5 cm rail, arm/home scripts
Rail
- Add firmware/rail_stepper/rail_stepper.ino (Arduino Uno, 115200 baud):
  limit switches lm_left (D5) and lm_right (D4), hardware stop at the
  switch in the direction of travel, calibration command "h"
  (lm_left -> lm_right -> middle -> 0), absolute moves "a<N>", and a
  50 Hz status line "ST <lm_left> <lm_right> <pos_steps> <homed>"
- rail_driver: background serial reader, ~/calibrate service, publishes
  /rail/position_cm, /rail/lm_left, /rail/lm_right at 50 Hz; position now
  comes from the Arduino and is measured from the left end; rejects rail
  goals until calibrated; aborts on move timeout instead of assuming done;
  warns if the calibrated length differs from expected_length_m
- Measured rail travel 71.5 cm: rail_joint limits 0.0-0.715 m in URDF,
  MoveIt joint_limits, GUI, mock and example scripts; rail_zero_x centres
  the travel on the 1 m rail mesh

Arm
- Add go_home (saved home pose read from the real arm; rail home prepared
  but commented out), arm_reach_grip and rail_reach_grip examples
- tools/example: wrap ROS setup sourcing in set +u

Docs
- README: port detection and --port/--rail-port, go home first, rail
  calibration on every bringup, things to know

Co-Authored-By: Claude Opus 5.5 <noreply@anthropic.com>

File: src/lerobot_description/urdf/so101_base.xacro (robot description, xacro)
@@ -12,6 +12,12 @@
 		needs to be changed when the rail alignment is corrected.
 	-->
-	<xacro:arg name="rail_lower" default="-0.5" />
-	<xacro:arg name="rail_upper" default="0.5" />
+	<!--
+		rail_joint = 0 is the left end (lm_left switch), increasing towards
+		lm_right. Measured travel between the switches: 71.5 cm. The travel is
+		centred on the 1 m rail mesh, so 0 sits at world x = -0.3575.
+	-->
+	<xacro:arg name="rail_lower" default="0.0" />
+	<xacro:arg name="rail_upper" default="0.715" />
+	<xacro:arg name="rail_zero_x" default="-0.3575" />
 	<xacro:arg name="rail_velocity" default="1.0" />
 	<xacro:arg name="rail_mount_x" default="-0.03" />
@@ -80,5 +86,5 @@
 		<parent link="rail_link" />
 		<child link="carriage_link" />
-		<origin xyz="0 0 0" rpy="0 0 0" />
+		<origin xyz="$(arg rail_zero_x) 0 0" rpy="0 0 0" />
 		<axis xyz="1 0 0" />
 		<limit effort="50" velocity="$(arg rail_velocity)"
